File: PCB/Rev1.0/AT-ProtoKeeb_rev1/AT-ProtoKeeb_rev1.kicad_pcb (KiCad board)
At the start: 2 copper layers, 80.2 x 99 mm, 112 parts, among them J1 USB4105-GF-A, U1 Raspberry Pi Pico, U2 TXB0102DCU, U3 USBLC6-2SC6

Commit message: minor changes and improvements in the Protokeeb Rev1 PCB files
Parts:
- added JP2: ARGB LED Data Link, Jumper:SolderJumper-2_P1.3mm_Open_TrianglePad1.0x1.5mm, F.Cu at (69.2, 58.7)
- added JP3: ARGB LED Data Link, Jumper:SolderJumper-2_P1.3mm_Open_TrianglePad1.0x1.5mm, F.Cu at (66.0, 58.7)
- U2: value TXB0102DCU -> TXB0102DCUR; footprint Package_SO:VSSOP-8_2.4x2.1mm_P0.5mm -> TXB0102DCUR:SOP50P310X90-8N
- U3: footprint Package_TO_SOT_SMD:SOT-23-6 -> USBLC6-2SC6:SOT95P280X145-6N
Routing:
- net Neopixel-2: track 6.29 -> 28.4 mm, vias 1 -> 2
- net Neopixel-1: track 6.23 -> 23.2 mm, vias 1 -> 3
- net DATA-IN-1: track 89.8 -> 94.8 mm, vias 6 -> 8
- net Net-(U2-OE): track 17.9 -> 13.3 mm, vias 2 -> 0
- net DATA-IN-2: track 148.1 -> 150.2 mm
